File: Hardware/board.brd (EAGLE design)
At the start: 46 x 35 mm, 105 parts, among them IC1 BQ25180YBGR, IC2 DRV2605YZFR, IC3 BMA421, IC9 RT6160AWSC, J1 503480-2400, J2 TC2030-IDC, J4 KH-TYPE-C-16P, Q1 DMG2305UX-7, Q3 SI1308EDL-T1-GE3, U1 NRF52840_QF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

Commit message: schematic corectat + board
Parts:
- moved TP_SWDCLK 223.9 mm to (19.3, -14.7)
- moved C34 222.2 mm to (5.97, -11.3)
- moved TP_OP 213.6 mm to (8.38, -10.5)
- moved TP_ON 213.4 mm to (6.73, -17.0)
- moved C23 208.7 mm to (9.53, 4.95), turned to 270 degrees
- moved C42 203.2 mm to (3.56, 13.7), turned to 90 degrees
- moved ANT1 202.4 mm to (-17.8, -12.7), turned to 180 degrees
- moved TP_3V3 200.9 mm to (8.51, -5.84)
- moved TP_SCL 197.5 mm to (16.0, -1.78)
- moved C21 196.1 mm to (-2.79, -6.22), turned to 90 degrees
- moved R7 195.6 mm to (13.8, -16.1), turned to 90 degrees
- moved IC3 195.6 mm to (19.7, -0.76)
- moved C20 193.6 mm to (-0.76, -6.35), turned to 90 degrees
- moved Q3 193.4 mm to (20.1, 12.5), turned to 90 degrees
- moved C43 191.6 mm to (3.68, 10.9), turned to 90 degrees
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Connections:
- net P0.03 renamed P1.03
- net P0.05 renamed P1.05
- net P0.06 renamed P1.06
- net P0.07 renamed P1.07
- removed net P0.02: U1.P$W24
- new net P1.04: U1.P$U24
- net N$10: now also U1.P$A23
- net P0.01: no longer U1.P$Y23
- net P0.04: no longer U1.P$U24
- net P1.01: now also U1.P$Y23
- net P1.02: now also U1.P$W24
Routing:
- net SDA: track 0.00 -> 81.8 mm, vias 0 -> 7
- net SCL: track 0.00 -> 73.8 mm, vias 0 -> 4
- net GND: track 0.00 -> 35.0 mm, vias 0 -> 16
- net IMU_INT1: track 0.00 -> 33.8 mm, vias 0 -> 2
- net IMU_INT2: track 0.00 -> 31.4 mm, vias 0 -> 2
- net SWDCLK: track 0.00 -> 29.0 mm, vias 0 -> 2
- net N$10: track 0.00 -> 28.9 mm, vias 0 -> 2
- net 3V3: track 0.00 -> 26.4 mm, vias 0 -> 8
- net PMIC_INT: track 0.00 -> 25.6 mm, vias 0 -> 2
- net P1.02: track 0.00 -> 25.2 mm, vias 0 -> 2
- net P1.01: track 0.00 -> 25.1 mm, vias 0 -> 2
- net MOSI: track 0.00 -> 24.6 mm, vias 0 -> 4
- net SWDIO: track 0.00 -> 20.3 mm
- net DEC4_6: track 0.00 -> 20.1 mm, vias 0 -> 2
- net SCK: track 0.00 -> 19.0 mm, vias 0 -> 3
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- added copper zone on layer 15, net 3V3
- added copper zone on layer 2, net GND
